Commit message: Adjusting demo for gripper

File: urdf/egp50.urdf.xacro (robot description, xacro)
@@ -25,5 +25,15 @@
 	<material name="blue"/>
       </collision>
+      <inertial>
+	<mass value="0.51" />
+ 	<inertia ixx="0.0007" iyy="0.0001" izz="0.0006" ixy="0.0" ixz="0.0" iyz="0.0" />
+      </inertial>
     </link>
+    <link name="egp_50_tip" />
+    <joint name="egp50_tip_joint" type="fixed">
+	<parent link="egp50_base_link"/>
+	<child link="egp_50_tip" />
+	<origin xyz="0.0 0.0 ${height}" rpy="0.0 0.0 0.0" />
+    </joint>
   </xacro:macro>
 </robot>

Commit message: Upgrade URDF

File: urdf/egp50.urdf.xacro (robot description, xacro)
@@ -1,27 +1,54 @@
 <?xml version="1.0"?>
-<robot xmlns:xacro="http://www.ros.org/wiki/xacro">
+<robot xmlns:xacro="http://www.ros.org/wiki/xacro" name="egp50">
   <xacro:macro name="schunk_egp50">
 <!--GRIPPER-->
-   <xacro:property name="length" value="0.05" />
-   <xacro:property name="width" value="0.03" />
-   <xacro:property name="height" value="0.118" />
+<!-- Base plate has 75mm diameter, 15mm thickness. Gripper body has 115mm height + pincers have 15mm height-->
+   <xacro:property name="base_diamter" value="0.075" />
+   <xacro:property name="base_length" value="0.015" />
+   <xacro:property name="body_length" value="0.05" />
+   <xacro:property name="body_width" value="0.03" />
+   <xacro:property name="body_height" value="0.115" />
+   <xacro:property name="pincer_height" value="0.015" />
+   <material name="blue">
+     <color rgba="0 0 1 1"/>
+   </material>
+    <material name="green">
+      <color rgba="0 1 0 1"/>
+    </material>
+    <material name="white">
+      <color rgba="1 1 1 1"/>
+    </material>
+    <!--Base plate-->
     <link name="egp50_base_link">
       <visual>
         <geometry>
+          <cylinder length="${base_length}" radius="${base_diamter/2}"/>
+        </geometry>
+        <material name="blue"/>
+        <origin rpy="0 0 0" xyz="0 0 ${base_length/2}"/>
+      </visual>
+      <collision>
+        <geometry>
+          <cylinder length="${base_length}" radius="${base_diamter/2}"/>
+        </geometry>
+        <origin rpy="0 0 0" xyz="0 0 0"/>
+      </collision>
+    </link>
+    <!--Main gripper-->
+    <link name="egp50_body_link">
+      <visual>
+        <geometry>
  	  <!--mesh filename="$(find ur_manipulation)/meshes/EGP50.stl" /-->
-	  <box size="${length} ${width} ${height}" />
+          <box size="${body_length} ${body_width} ${body_height}" />
         </geometry>
-	<origin rpy="0 0 0" xyz="0 0 0.059"/>
-        <material name="blue">
-          <color rgba="0 0 1 1"/>
-        </material>
+        <material name="green"/>
+        <origin rpy="0 0 0" xyz="0 0 0"/>
       </visual>
       <collision>
         <geometry>
           <!--mesh filename="$(find ur_manipulation)/meshes/EGP50.stl" /-->
-	  <box size="${length} ${width} ${height}" />
+          <box size="${body_length} ${body_width} ${body_height}" />
         </geometry>
-	<origin rpy="0 0 0" xyz="0 0 0.059"/>
-	<material name="blue"/>
+        <origin rpy="0 0 0" xyz="0 0 0"/>
       </collision>
       <inertial>
@@ -30,9 +57,41 @@
       </inertial>
     </link>
+    <!--Pincer block-->
+    <link name="egp50_pincer_link">
+      <visual>
+        <geometry>
+          <box size="${body_length} ${body_width} ${pincer_height}" />
+        </geometry>
+        <origin rpy="0 0 0" xyz="0 0 0"/>
+        <material name="white"/>
+      </visual>
+      <collision>
+        <geometry>
+          <box size="${body_length} ${body_width} ${pincer_height}" />
+        </geometry>
+        <origin rpy="0 0 0" xyz="0 0 0"/>
+      </collision>
+      <inertial>
+        <mass value="0.51" />
+        <inertia ixx="0.0007" iyy="0.0001" izz="0.0006" ixy="0.0" ixz="0.0" iyz="0.0" />
+      </inertial>
+    </link>
+    <!-- Virtual link for visualizytion and planning-->
     <link name="egp_50_tip" />
+   <!-- Joints-->
+    <joint name="egp50_body_joint" type="fixed">
+        <parent link="egp50_base_link"/>
+        <child link="egp50_body_link" />
+        <origin xyz="0.0 0.0 ${base_length+body_height/2}" rpy="0.0 0.0 0.0" />
+    </joint>
+    <joint name="egp50_pincer_joint" type="fixed">
+        <parent link="egp50_body_link"/>
+        <child link="egp50_pincer_link" />
+        <origin xyz="0.0 0.0 ${body_height/2+pincer_height/2}" rpy="0.0 0.0 0.0" />
+    </joint>
     <joint name="egp50_tip_joint" type="fixed">
-	<parent link="egp50_base_link"/>
+        <parent link="egp50_pincer_link"/>
 	<child link="egp_50_tip" />
-	<origin xyz="0.0 0.0 ${height}" rpy="0.0 0.0 0.0" />
+        <origin xyz="0.0 0.0 ${pincer_height/2}" rpy="0.0 0.0 0.0" />
     </joint>
   </xacro:macro>

Commit message: Benchmarking mqtt changes

File: urdf/egp50.urdf.xacro (robot description, xacro)
@@ -72,8 +72,8 @@
         <origin rpy="0 0 0" xyz="0 0 0"/>
       </collision>
-      <inertial>
+      <!--inertial>
         <mass value="0.51" />
         <inertia ixx="0.0007" iyy="0.0001" izz="0.0006" ixy="0.0" ixz="0.0" iyz="0.0" />
-      </inertial>
+      </inertial-->
     </link>
     <!-- Virtual link for visualizytion and planning-->
